File: Group_project_5/Kicad_files/motorcontroller/motorcontroller.sch (KiCad schematic (older format))
At the start: 12 parts, among them J1 Raspberry_Pi_2_3, J2 Arduino_Nano_Every, J3 Arduino_Nano_Every, SW1 SW_DIP_x02, U1 Logic_Level_Shifter

Commit message: Fixed pcb
Parts:
- SW1: footprint Button_Switch_SMD:SW_DIP_SPSTx02_Slide_6.7x6.64mm_W6.73mm_P2.54mm_LowProfile_JPin -> Button_Switch_SMD:SW_DIP_SPSTx02_Slide_6.7x6.64mm_W8.61mm_P2.54mm_LowProfile
Connections:
- net +5V: now also J2.27 (+5V), J3.27 (+5V); no longer J2.30 (VIN), J3.30 (VIN)
- net at J2.2 (RX1): now also SW1.4; no longer SW1.3
- net at J3.2 (RX1): now also SW1.3; no longer SW1.4
Changed lines of the file:
@@
 L power:+5V #PWR0103
 U 1 1 617FB7F9
-P 6550 1450
-F 0 "#PWR0103" H 6550 1300 50  0001 C CNN
-F 1 "+5V" H 6565 1623 50  0000 C CNN
-F 2 "" H 6550 1450 50  0001 C CNN
-F 3 "" H 6550 1450 50  0001 C CNN
-	1    6550 1450
+P 6850 1450
+F 0 "#PWR0103" H 6850 1300 50  0001 C CNN
+F 1 "+5V" H 6865 1623 50  0000 C CNN
+F 2 "" H 6850 1450 50  0001 C CNN
+F 3 "" H 6850 1450 50  0001 C CNN
+	1    6850 1450
 	1    0    0    -1
 $EndComp
@@
 L power:+5V #PWR0104
 U 1 1 61802F8C
-P 9000 1450
-F 0 "#PWR0104" H 9000 1300 50  0001 C CNN
-F 1 "+5V" H 9015 1623 50  0000 C CNN
-F 2 "" H 9000 1450 50  0001 C CNN
-F 3 "" H 9000 1450 50  0001 C CNN
-	1    9000 1450
+P 9300 1450
+F 0 "#PWR0104" H 9300 1300 50  0001 C CNN
+F 1 "+5V" H 9315 1623 50  0000 C CNN
+F 2 "" H 9300 1450 50  0001 C CNN
+F 3 "" H 9300 1450 50  0001 C CNN
+	1    9300 1450
 	1    0    0    -1
 $EndComp
@@
 	3300 6700 3200 6700
 Wire Wire Line
-	6550 1450 6550 1500
-Wire Wire Line
-	9000 1450 9000 1500
+	6850 1450 6850 1500
+Wire Wire Line
+	9300 1450 9300 1500
 Text GLabel 6050 3000 0    50   Input ~ 0
 PWM_Pin_0_Left
@@
 F 0 "SW1" H 5500 1667 50  0000 C CNN
 F 1 "SW_DIP_x02" H 5500 1576 50  0000 C CNN
-F 2 "Button_Switch_SMD:SW_DIP_SPSTx02_Slide_6.7x6.64mm_W6.73mm_P2.54mm_LowProfile_JPin" H 5500 1300 50  0001 C CNN
+F 2 "Button_Switch_SMD:SW_DIP_SPSTx02_Slide_6.7x6.64mm_W8.61mm_P2.54mm_LowProfile" H 5500 1300 50  0001 C CNN
 F 3 "~" H 5500 1300 50  0001 C CNN
 	1    5500 1300
@@
 Wire Wire Line
 	5100 1200 5200 1200
-Wire Wire Line
-	5800 1200 8400 1200
-Wire Wire Line
-	5800 1300 5900 1300
-Wire Wire Line
-	5900 1300 5900 1800
 Wire Wire Line
 	5000 1450 5000 1550
@@
 Wire Wire Line
 	8600 2050 8600 2100
+Wire Wire Line
+	5900 1200 5800 1200
+Wire Wire Line
+	5900 1200 5900 1800
+Wire Wire Line
+	5800 1300 6050 1300
+Wire Wire Line
+	6050 1300 6050 1200
+Wire Wire Line
+	6050 1200 8400 1200
 $EndSCHEMATC
