File: Group_project_5/Kicad_files/motorcontroller/Motor&Power.sch (KiCad schematic (older format))
At the start: 6 parts, among them J6 Battery_Connector, J7 Motor_Left, J8 Motor_Right, SW2 SW_SPDT, U2 DC-DCXL6009E1, U3 DRV8833_breakout_board

Commit message: Fixed pcb
Connections:
- net at J8.1 (Pin_1): now also U3.4 (BOUT1); no longer U3.3 (BOUT2)
- net at J8.6 (Pin_6): now also U3.3 (BOUT2); no longer U3.4 (BOUT1)
Changed lines of the file:
@@
 	2600 2400 3450 2400
 Wire Wire Line
-	3450 2500 3300 2500
-Wire Wire Line
-	3300 2500 3300 4150
-Wire Wire Line
 	3300 4150 1900 4150
-Wire Wire Line
-	3450 2600 3250 2600
-Wire Wire Line
-	3250 2600 3250 3650
 Wire Wire Line
 	3250 3650 1900 3650
@@
 	0    1    1    0
 $EndComp
+Wire Wire Line
+	3250 2500 3250 3650
+Wire Wire Line
+	3250 2500 3450 2500
+Wire Wire Line
+	3300 4150 3300 2600
+Wire Wire Line
+	3300 2600 3450 2600
 $EndSCHEMATC
