File: Group_project_5/Kicad_files/motorcontroller/motorcontroller.kicad_pcb (KiCad board)
At the start: 2 copper layers, 133.7 x 90.8 mm, 22 parts, among them J1 Raspberry_Pi_2_3, J2 Arduino_Nano_Every, J3 Arduino_Nano_Every, J4 Conn_01x03, J5 Conn_01x03, J6 Battery_Connector, J7 Motor_Left, J8 Motor_Right, SW1 SW_DIP_x02, SW2 SW_SPDT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

Commit message: Fixed pcb
Parts:
- added REF**: PinHeader_1x01_P2.54mm_Vertical, Connector_PinHeader_2.54mm:PinHeader_1x01_P2.54mm_Vertical, F.Cu at (167.3, 112.7)
- added REF**: PinHeader_1x01_P2.54mm_Vertical, Connector_PinHeader_2.54mm:PinHeader_1x01_P2.54mm_Vertical, F.Cu at (105.1, 104.8)
- added REF**: PinHeader_1x01_P2.54mm_Vertical, Connector_PinHeader_2.54mm:PinHeader_1x01_P2.54mm_Vertical, F.Cu at (173.8, 96.5)
- added REF**: PinHeader_1x01_P2.54mm_Vertical, Connector_PinHeader_2.54mm:PinHeader_1x01_P2.54mm_Vertical, F.Cu at (111.7, 113.1)
- added REF**: PinHeader_1x01_P2.54mm_Vertical, Connector_PinHeader_2.54mm:PinHeader_1x01_P2.54mm_Vertical, F.Cu at (88.6, 113.8)
- added REF**: PinHeader_1x01_P2.54mm_Vertical, Connector_PinHeader_2.54mm:PinHeader_1x01_P2.54mm_Vertical, F.Cu at (99.3, 101.6)
- added REF**: PinHeader_1x01_P2.54mm_Vertical, Connector_PinHeader_2.54mm:PinHeader_1x01_P2.54mm_Vertical, F.Cu at (165.5, 120.2)
- added REF**: PinHeader_1x01_P2.54mm_Vertical, Connector_PinHeader_2.54mm:PinHeader_1x01_P2.54mm_Vertical, F.Cu at (164.8, 107.2)
- added REF**: PinHeader_1x01_P2.54mm_Vertical, Connector_PinHeader_2.54mm:PinHeader_1x01_P2.54mm_Vertical, F.Cu at (130.4, 80.6)
- added REF**: PinHeader_1x01_P2.54mm_Vertical, Connector_PinHeader_2.54mm:PinHeader_1x01_P2.54mm_Vertical, F.Cu at (168.3, 125.5)
- SW1: footprint Button_Switch_SMD:SW_DIP_SPSTx02_Slide_6.7x6.64mm_W6.73mm_P2.54mm_LowProfile_JPin -> Button_Switch_SMD:SW_DIP_SPSTx02_Slide_6.7x6.64mm_W8.61mm_P2.54mm_LowProfile
- moved SW2 1.85 mm to (150.7, 100.3)
- moved J7 1.52 mm to (102.6, 117.2)
- moved J8 1.34 mm to (90.0, 91.4)
- moved J5 0.76 mm to (165.5, 92.0)
- moved U2 0.63 mm to (145.9, 115.2)
- moved SW1 0.13 mm to (152.3, 113.1)
Connections:
- J2 pad 27: Net-(J2-Pad27) -> +5V
- J2 pad 30: +5V -> Net-(J2-Pad30)
- J3 pad 27: Net-(J3-Pad27) -> +5V
- J3 pad 30: +5V -> Net-(J3-Pad30)
- REF** pad 1: (no net) -> GND (x2)
- U3 pad 3: Net-(J8-Pad1) -> Net-(J8-Pad6)
- U3 pad 4: Net-(J8-Pad6) -> Net-(J8-Pad1)
Routing:
- net +5V: track 234.6 -> 290.4 mm
- net +3V3: track 33.9 -> 76.9 mm
- net PWM_Pin_1_Right: track 40.2 -> 65.6 mm
- net PWM_Pin_0_Right: track 39.4 -> 62.2 mm
- net FLT: track 28.6 -> 12.4 mm
- net Net-(D1-Pad2): track 31.6 -> 45.2 mm
- net Net-(J7-Pad6): track 24.4 -> 34.9 mm
- net FLT_pi: track 8.82 -> 18.1 mm
- net Net-(J8-Pad6): track 16.5 -> 25.6 mm
- net PWM_Pin_0_Left: track 60.3 -> 51.6 mm
- net PWM_Pin_1_Left: track 54.6 -> 46.1 mm
- net Net-(J2-Pad2): track 20.5 -> 26.5 mm
- net Net-(J7-Pad1): track 34.5 -> 30.1 mm
- net Net-(J8-Pad1): track 9.06 -> 6.70 mm
- net Net-(J6-Pad2): track 9.70 -> 7.72 mm
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- removed copper zone on B.Cu, net GND
Other:
- board size 133.7 x 90.8 mm -> 111.6 x 90.8 mm
- rule trace_min: 0.2 -> 0.254
- rule via_min_size: 0.4 -> 1

Commit message: yaddaydda
Changed lines of the file:
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@@
     (thickness 1.6)
     (drawings 44)
-    (tracks 184)
+    (tracks 185)
     (zones 0)
     (modules 32)
@@
     (mod_text_size 1 1)
     (mod_text_width 0.15)
-    (pad_size 1.8 1.8)
+    (pad_size 1.6 1.6)
     (pad_drill 1)
     (pad_to_mask_clearance 0)
@@
     (fp_arc (start 1.27 0) (end -0.29 -1.235516) (angle 108.8) (layer F.SilkS) (width 0.12))
     (fp_arc (start 1.27 0) (end -0.23 -1.16619) (angle 284.3) (layer F.Fab) (width 0.1))
-    (pad 2 thru_hole circle (at 2.54 0 90) (size 1.8 1.8) (drill 1) (layers *.Cu *.Mask)
+    (pad 2 thru_hole circle (at 2.54 0 90) (size 1.7 1.7) (drill 1) (layers *.Cu *.Mask)
       (net 3 "Net-(D2-Pad2)"))
-    (pad 1 thru_hole rect (at 0 0 90) (size 1.8 1.8) (drill 1) (layers *.Cu *.Mask)
+    (pad 1 thru_hole circle (at 0 0 90) (size 1.7 1.7) (drill 1) (layers *.Cu *.Mask)
       (net 4 "Net-(D2-Pad1)"))
     (model ${KISYS3DMOD}/LED_THT.3dshapes/LED_D3.0mm.wrl
@@
       (effects (font (size 1 1) (thickness 0.15)))
     )
-    (pad 2 thru_hole oval (at 10.16 0 270) (size 1.8 1.8) (drill 0.9) (layers *.Cu *.Mask)
+    (pad 2 thru_hole oval (at 10.16 0 270) (size 1.8 1.8) (drill 1) (layers *.Cu *.Mask)
       (net 5 "Net-(D3-Pad2)"))
     (pad 1 thru_hole rect (at 0 0 270) (size 1.8 1.8) (drill 1) (layers *.Cu *.Mask)
@@
   (segment (start 169.1005 97.2185) (end 169.6085 97.2185) (width 0.254) (layer F.Cu) (net 85))
   (segment (start 177.673 111.4425) (end 177.9905 111.4425) (width 0.254) (layer F.Cu) (net 86))
-  (segment (start 174.244 108.0135) (end 177.673 111.4425) (width 0.508) (layer F.Cu) (net 86))
-  (segment (start 174.244 104.267) (end 174.244 108.0135) (width 0.508) (layer F.Cu) (net 86))
+  (segment (start 177.292 111.4425) (end 177.673 111.4425) (width 0.508) (layer F.Cu) (net 86))
+  (segment (start 174.244 108.3945) (end 177.292 111.4425) (width 0.508) (layer F.Cu) (net 86))
+  (segment (start 174.244 104.267) (end 174.244 108.3945) (width 0.508) (layer F.Cu) (net 86))
   (segment (start 171.069 101.092) (end 174.244 104.267) (width 0.508) (layer F.Cu) (net 86))
   (segment (start 169.4815 101.092) (end 171.069 101.092) (width 0.508) (layer F.Cu) (net 86))
